Commit message: Submission Draft

File: src/my_robot/urdf/my_robot.xacro (robot description, xacro)
@@ -9,12 +9,12 @@
   </joint>
   <link name='chassis'>
-    <pose>0 0 0.1 0 0 0</pose>
+    <pose>0 0 0.4 0 0 0</pose>
     <inertial>
       <mass value="15.0"/>
       <origin xyz="0.0 0 0" rpy=" 0 0 0"/>
       <inertia
-          ixx="0.1" ixy="0" ixz="0"
-          iyy="0.1" iyz="0"
-          izz="0.1"
+          ixx="0.3" ixy="0" ixz="0"
+          iyy="0.3" iyz="0"
+          izz="0.3"
       />
     </inertial>
@@ -22,5 +22,5 @@
       <origin xyz="0 0 0" rpy=" 0 0 0"/>
       <geometry>
-        <box size=".4 .2 .1"/>
+        <box size=".6 .8 .4"/>
       </geometry>
     </collision>
@@ -28,29 +28,45 @@
       <origin xyz="0 0 0" rpy=" 0 0 0"/>
       <geometry>
-        <box size=".4 .2 .1"/>
+        <box size=".8 .8 .4"/>
       </geometry>
     </visual>
     <collision name='back_caster_collision'>
-      <origin xyz="-0.15 0 -0.05" rpy=" 0 0 0"/>
+      <origin xyz="-0.25 0 -0.2" rpy=" 0 0 0"/>
       <geometry>
-        <sphere radius="0.0499"/>
+        <sphere radius="0.14"/>
       </geometry>
+      <surface>
+        <friction>
+          <ode>
+            <mu>0.0</mu>
+            <mu1>0.0</mu1>
+          </ode>
+        </friction>
+      </surface>
     </collision>
     <visual name='back_caster_visual'>
-      <origin xyz="-0.15 0 -0.05" rpy=" 0 0 0"/>
+      <origin xyz="-0.25 0 -0.2" rpy=" 0 0 0"/>
       <geometry>
-        <sphere radius="0.05"/>
+        <sphere radius="0.14"/>
       </geometry>
     </visual>
     <collision name='front_caster_collision'>
-      <origin xyz="0.15 0 -0.05" rpy=" 0 0 0"/>
+      <origin xyz="0.25 0 -0.2" rpy=" 0 0 0"/>
       <geometry>
-        <sphere radius="0.0499"/>
+        <sphere radius="0.14"/>
       </geometry>
+      <surface>
+        <friction>
+          <ode>
+            <mu>0.0</mu>
+            <mu1>0.0</mu1>
+          </ode>
+        </friction>
+      </surface>
     </collision>
     <visual name='front_caster_visual'>
-      <origin xyz="0.15 0 -0.05" rpy=" 0 0 0"/>
+      <origin xyz="0.25 0 -0.2" rpy=" 0 0 0"/>
       <geometry>
-        <sphere radius="0.05"/>
+        <sphere radius="0.14"/>
       </geometry>
     </visual>
@@ -60,5 +76,5 @@
       <origin xyz="0 0 0" rpy="0 1.5707 1.5707" />
       <geometry>
-      <cylinder radius="0.1" length="0.05" />
+      <cylinder radius="0.35" length="0.15" />
       </geometry>
     </collision>
@@ -66,5 +82,5 @@
       <origin xyz="0 0 0" rpy="0 1.5707 1.5707" />
       <geometry>
-      <cylinder radius="0.1" length="0.05" />
+      <cylinder radius="0.35" length="0.15" />
       </geometry>
     </visual>
@@ -73,12 +89,12 @@
       <origin xyz="0 0 0" rpy="0 1.5707 1.5707" />
       <inertia
-          ixx="0.1" ixy="0" ixz="0"
-          iyy="0.1" iyz="0"
-          izz="0.1"
+          ixx="0.3" ixy="0" ixz="0"
+          iyy="0.3" iyz="0"
+          izz="0.3"
       />
     </inertial>
   </link>
   <joint type="continuous" name="left_wheel_hinge">
-    <origin xyz="0 0.15 0" rpy="0 0 0"/>
+    <origin xyz="0 0.55 0" rpy="0 0 0"/>
     <child link="left_wheel"/>
     <parent link="chassis"/>
@@ -91,5 +107,5 @@
       <origin xyz="0 0 0" rpy="0 1.5707 1.5707" />
       <geometry>
-      <cylinder radius="0.1" length="0.05" />
+      <cylinder radius="0.35" length="0.15" />
       </geometry>
     </collision>
@@ -97,5 +113,5 @@
       <origin xyz="0 0 0" rpy="0 1.5707 1.5707" />
       <geometry>
-      <cylinder radius="0.1" length="0.05" />
+      <cylinder radius="0.35" length="0.15" />
       </geometry>
     </visual>
@@ -104,12 +120,12 @@
       <origin xyz="0 0 0" rpy="0 1.5707 1.5707" />
       <inertia
-          ixx="0.1" ixy="0" ixz="0"
-          iyy="0.1" iyz="0"
-          izz="0.1"
+          ixx="0.3" ixy="0" ixz="0"
+          iyy="0.3" iyz="0"
+          izz="0.3"
       />
     </inertial>
   </link>
   <joint type="continuous" name="right_wheel_hinge">
-    <origin xyz="0 -0.15 0" rpy="0 0 0"/>
+    <origin xyz="0 -0.55 0" rpy="0 0 0"/>
     <child link="right_wheel"/>
     <parent link="chassis"/>
@@ -142,5 +158,5 @@
   </link>
   <joint type="fixed" name="camera_joint">
-    <origin xyz="0.2 0 0" rpy="0 0 0 " />
+    <origin xyz="0.5 0 0.2" rpy="0 0 0 " />
     <axis xyz="0 1 0" rpy="0 0 0" />
     <parent link="chassis" />
@@ -171,5 +187,5 @@
   </link>
   <joint type="fixed" name="hokuyo_joint">
-    <origin xyz="0.15 0 0.1" rpy="0 0 0" />
+    <origin xyz="0.15 0 0.4" rpy="0 0 0" />
     <axis xyz="0 1 0" rpy="0 0 0" />
     <parent link="chassis" />

Commit message: Added teleop package. Changed world to be more interesting. Reduced Robot size.

File: src/my_robot/urdf/my_robot.xacro (robot description, xacro)
@@ -22,5 +22,5 @@
       <origin xyz="0 0 0" rpy=" 0 0 0"/>
       <geometry>
-        <box size=".6 .8 .4"/>
+        <box size=".2 .2 .1"/>
       </geometry>
     </collision>
@@ -28,11 +28,11 @@
       <origin xyz="0 0 0" rpy=" 0 0 0"/>
       <geometry>
-        <box size=".8 .8 .4"/>
+        <box size=".2 .2 .1"/>
       </geometry>
     </visual>
     <collision name='back_caster_collision'>
-      <origin xyz="-0.25 0 -0.2" rpy=" 0 0 0"/>
+      <origin xyz="-0.0625 0 -0.05" rpy=" 0 0 0"/>
       <geometry>
-        <sphere radius="0.14"/>
+        <sphere radius="0.035"/>
       </geometry>
       <surface>
@@ -46,13 +46,13 @@
     </collision>
     <visual name='back_caster_visual'>
-      <origin xyz="-0.25 0 -0.2" rpy=" 0 0 0"/>
+      <origin xyz="-0.0625 0 -0.05" rpy=" 0 0 0"/>
       <geometry>
-        <sphere radius="0.14"/>
+        <sphere radius="0.035"/>
       </geometry>
     </visual>
     <collision name='front_caster_collision'>
-      <origin xyz="0.25 0 -0.2" rpy=" 0 0 0"/>
+      <origin xyz="0.0625 0 -0.05" rpy=" 0 0 0"/>
       <geometry>
-        <sphere radius="0.14"/>
+        <sphere radius="0.035"/>
       </geometry>
       <surface>
@@ -66,7 +66,7 @@
     </collision>
     <visual name='front_caster_visual'>
-      <origin xyz="0.25 0 -0.2" rpy=" 0 0 0"/>
+      <origin xyz="0.0625 0 -0.05" rpy=" 0 0 0"/>
       <geometry>
-        <sphere radius="0.14"/>
+        <sphere radius="0.035"/>
       </geometry>
     </visual>
@@ -76,5 +76,5 @@
       <origin xyz="0 0 0" rpy="0 1.5707 1.5707" />
       <geometry>
-      <cylinder radius="0.35" length="0.15" />
+      <cylinder radius="0.0875" length="0.0375" />
       </geometry>
     </collision>
@@ -82,5 +82,5 @@
       <origin xyz="0 0 0" rpy="0 1.5707 1.5707" />
       <geometry>
-      <cylinder radius="0.35" length="0.15" />
+      <cylinder radius="0.0875" length="0.0375" />
       </geometry>
     </visual>
@@ -96,5 +96,5 @@
   </link>
   <joint type="continuous" name="left_wheel_hinge">
-    <origin xyz="0 0.55 0" rpy="0 0 0"/>
+    <origin xyz="0 0.1375 0" rpy="0 0 0"/>
     <child link="left_wheel"/>
     <parent link="chassis"/>
@@ -107,5 +107,5 @@
       <origin xyz="0 0 0" rpy="0 1.5707 1.5707" />
       <geometry>
-      <cylinder radius="0.35" length="0.15" />
+      <cylinder radius="0.0875" length="0.0375" />
       </geometry>
     </collision>
@@ -113,5 +113,5 @@
       <origin xyz="0 0 0" rpy="0 1.5707 1.5707" />
       <geometry>
-      <cylinder radius="0.35" length="0.15" />
+      <cylinder radius="0.0875" length="0.0375" />
       </geometry>
     </visual>
@@ -127,5 +127,5 @@
   </link>
   <joint type="continuous" name="right_wheel_hinge">
-    <origin xyz="0 -0.55 0" rpy="0 0 0"/>
+    <origin xyz="0 -0.1375 0" rpy="0 0 0"/>
     <child link="right_wheel"/>
     <parent link="chassis"/>
@@ -158,5 +158,5 @@
   </link>
   <joint type="fixed" name="camera_joint">
-    <origin xyz="0.5 0 0.2" rpy="0 0 0 " />
+    <origin xyz="0.125 0 0.05" rpy="0 0 0 " />
     <axis xyz="0 1 0" rpy="0 0 0" />
     <parent link="chassis" />
@@ -187,5 +187,5 @@
   </link>
   <joint type="fixed" name="hokuyo_joint">
-    <origin xyz="0.15 0 0.4" rpy="0 0 0" />
+    <origin xyz="0.0375 0 0.1" rpy="0 0 0" />
     <axis xyz="0 1 0" rpy="0 0 0" />
     <parent link="chassis" />

Commit message: editted world a little

File: src/my_robot/urdf/my_robot.xacro (robot description, xacro)
@@ -134,5 +134,5 @@
     <dynamics damping="1.0" friction="1.0"/>
   </joint>
-  <link name="camera">
+  <link name="camera_link">
     <visual name="camera_visual">
       <origin xyz="0 0 0" rpy="0 0 0"/>
@@ -161,5 +161,5 @@
     <axis xyz="0 1 0" rpy="0 0 0" />
     <parent link="chassis" />
-    <child link="camera" />
+    <child link="camera_link" />
   </joint>
   <link name="hokuyo">
@@ -192,3 +192,10 @@
     <child link="hokuyo" />
   </joint>
+  <joint name="camera_optical_joint" type="fixed">
+    <origin xyz="0 0 0" rpy="-1.5707 0 -1.5707"/>
+    <parent link="camera_link"/>
+    <child link="camera_link_optical"/>
+  </joint>
+  <link name="camera_link_optical">
+  </link>
 </robot>
